File: project-TPS62933-breakout.kicad_pcb (KiCad board)
At the start: 4 copper layers, 36 x 23 mm, 14 parts, among them J1 Conn_01x04_Pin, U1 TPS7A2033PDBVR, U2 TPS62933DRLR

Commit message: pcb: update version
Other:
- board text added: "v1.0.0-9-gfdc2d40"
- board text removed: "v1.0.0-3-g22dea1a"
